File: keyboard-tutorial.kicad_pcb (KiCad board)
At the start: 2 copper layers, 84.1 x 38.1 mm, 24 parts, among them SW1 SW_Push, U1 ATmega32U4-A, Y1 16MHz

Commit message: Post Tracing
Parts:
- moved R2 1.59 mm to (56.4, 49.2)
- moved C5 1.59 mm to (68.3, 57.1), turned to 180 degrees
- turned C7 to -90 degrees
Routing:
- net GND: track 0.00 -> 112.0 mm
- net Net-(R3-Pad2): track 0.00 -> 48.5 mm
- net +5V: track 0.00 -> 41.4 mm
- net Net-(R2-Pad2): track 0.00 -> 35.1 mm
- net Net-(R4-Pad2): track 0.00 -> 30.7 mm
- net Net-(C7-Pad2): track 0.00 -> 23.2 mm
- net Net-(C6-Pad2): track 0.00 -> 13.8 mm
- net D-: track 0.00 -> 11.8 mm
- net VCC: track 0.00 -> 11.0 mm
- net Net-(R1-Pad1): track 0.00 -> 3.86 mm
